File: hw/PocketFT8Xcvr.kicad_pcb (KiCad board)
At the start: 4 copper layers, 0 parts

Commit message: Imported components to PCB
Parts:
- added BAT1: BU2032SM-JJ-GTR, BU2032SM:BU2032SM-JJ-GTR_MPD, F.Cu at (43.2, 45.7)
- added C1: 0.1UF, Capacitor_SMD:C_0603_1608Metric, F.Cu at (39.4, 57.8)
- added C10: 75PF, Capacitor_SMD:C_0805_2012Metric, F.Cu at (28.3, 76.1)
- added C11: 0.1UF, Capacitor_SMD:C_0603_1608Metric, F.Cu at (39.4, 65.4)
- added C12: 0.1UF, Capacitor_SMD:C_0603_1608Metric, F.Cu at (39.4, 67.9)
- added C13: 0.1UF, Capacitor_SMD:C_0603_1608Metric, F.Cu at (39.4, 70.4)
- added C14: 0.1UF, Capacitor_SMD:C_0603_1608Metric, F.Cu at (39.4, 72.9)
- added C15: 0.1UF, Capacitor_SMD:C_0603_1608Metric, F.Cu at (39.4, 75.4)
- added C16: 0.1UF, Capacitor_SMD:C_0603_1608Metric, F.Cu at (43.4, 57.8)
- added C17: 0.1UF, Capacitor_SMD:C_0603_1608Metric, F.Cu at (43.4, 60.3)
- added C18: 0.1UF, Capacitor_SMD:C_0603_1608Metric, F.Cu at (43.4, 62.9)
- added C19: 0.1UF, Capacitor_SMD:C_0603_1608Metric, F.Cu at (43.4, 65.4)
- added C2: 10UF, Capacitor_SMD:C_0805_2012Metric, F.Cu at (28.3, 58.1)
- added C20: 0.1UF, Capacitor_SMD:C_0603_1608Metric, F.Cu at (43.4, 67.9)
- added C21: 0.1UF, Capacitor_SMD:C_0603_1608Metric, F.Cu at (43.4, 70.4)
- added C22: 0.1UF, Capacitor_SMD:C_0603_1608Metric, F.Cu at (43.4, 72.9)
- added C23: 0.33UF, digikey-footprints:0805, F.Cu at (73.5, 82.8)
- added C24: 0.1UF, Capacitor_SMD:C_0603_1608Metric, F.Cu at (43.4, 75.4)
- added C25: 0.1UF, Capacitor_SMD:C_0603_1608Metric, F.Cu at (47.4, 57.8)
- added C26: 47PF, Capacitor_SMD:C_0805_2012Metric, F.Cu at (28.3, 79.2)
- added C3: 0.1UF, Capacitor_SMD:C_0603_1608Metric, F.Cu at (39.4, 60.3)
- added C4: 0.1UF, Capacitor_SMD:C_0603_1608Metric, F.Cu at (39.4, 62.9)
- added C5: 10UF, Capacitor_SMD:C_0805_2012Metric, F.Cu at (28.3, 61.1)
- added C6: 10UF, Capacitor_SMD:C_0805_2012Metric, F.Cu at (28.3, 64.1)
- added C7: 10UF, Capacitor_SMD:C_0805_2012Metric, F.Cu at (28.3, 67.1)
- added C8: 75PF, Capacitor_SMD:C_0805_2012Metric, F.Cu at (28.3, 70.1)
- added C9: 243PF, Capacitor_SMD:C_0805_2012Metric, F.Cu at (28.3, 73.1)
- added D1: XMIT, LED_THT:LED_D5.0mm, F.Cu at (73.5, 77.6)
- added J1: HX8357D, Connector_PinHeader_2.54mm:PinHeader_1x20_P2.54mm_Vertical, F.Cu at (198.1, 61.0)
- added J2: 22-23-2021, digikey-footprints:PinHeader_1x2_P2.54mm_Drill1.02mm, F.Cu at (60.1, 77.8)
- added J3: 22-23-2021, digikey-footprints:PinHeader_1x2_P2.54mm_Drill1.02mm, F.Cu at (66.5, 77.8)
- added J4: Conn_01x07, Connector_PinHeader_2.54mm:PinHeader_1x07_P2.54mm_Vertical, F.Cu at (55.8, 58.9)
- added J5: HX8357D, Connector_PinHeader_2.54mm:PinHeader_1x20_P2.54mm_Vertical, F.Cu at (106.7, 61.0)
- added L1: 0.5uH, Inductor_THT:L_Toroid_Vertical_L10.0mm_W5.0mm_P5.08mm, F.Cu at (63.9, 58.4)
- added L2: 0.5uH, Inductor_THT:L_Toroid_Vertical_L10.0mm_W5.0mm_P5.08mm, F.Cu at (63.9, 67.0)
- added L3: 1.0mH, footprints:IND_BOURNS_RLB9012, F.Cu at (41.1, 81.9)
- added Q1: 2N3904, digikey-footprints:TO-92-3, F.Cu at (32.7, 59.6)
- added Q2: 2N3906, digikey-footprints:TO-92-3, F.Cu at (32.7, 64.9)
- added Q3: 2N7000, digikey-footprints:TO-92-3, F.Cu at (32.7, 70.2)
- added Q4: 2N7000, digikey-footprints:TO-92-3, F.Cu at (32.7, 75.5)
- added R1: 2.0K, Resistor_SMD:R_0603_1608Metric, F.Cu at (47.4, 60.3)
- added R10: 5.1K, Resistor_SMD:R_0603_1608Metric, F.Cu at (51.4, 62.9)
- added R11: 510 Ohm, Resistor_SMD:R_0603_1608Metric, F.Cu at (51.4, 65.4)
- added R2: 2.0K, Resistor_SMD:R_0603_1608Metric, F.Cu at (47.4, 62.9)
- added R3: 47K, Resistor_SMD:R_0603_1608Metric, F.Cu at (47.4, 65.4)
- added R4: 47K, Resistor_SMD:R_0603_1608Metric, F.Cu at (47.4, 67.9)
- added R5: 2.0K, Resistor_SMD:R_0603_1608Metric, F.Cu at (47.4, 70.4)
- added R6: 10K, Resistor_SMD:R_0603_1608Metric, F.Cu at (47.4, 72.9)
- added R7: 51 OHM, Resistor_SMD:R_0603_1608Metric, F.Cu at (47.4, 75.4)
- added R8: 510 Ohm, Resistor_SMD:R_0603_1608Metric, F.Cu at (51.4, 57.8)
- added R9: 5.1K, Resistor_SMD:R_0603_1608Metric, F.Cu at (51.4, 60.3)
- added REF**: MountingHole_2.2mm_M2, MountingHole:MountingHole_2.2mm_M2, F.Cu at (106.7, 114.9)
- added REF**: MountingHole_2.2mm_M2, MountingHole:MountingHole_2.2mm_M2, F.Cu at (198.1, 54.0)
- added REF**: MountingHole_2.2mm_M2, MountingHole:MountingHole_2.2mm_M2, F.Cu at (198.1, 114.9)
- added REF**: MountingHole_2.2mm_M2, MountingHole:MountingHole_2.2mm_M2, F.Cu at (106.7, 54.0)
- added TN1: Teensy4.1, teensy:Teensy41, F.Cu at (123.2, 27.9)
- added U1: MCP3422A1T-E/SN, Package_SO:SOIC-8_3.9x4.9mm_P1.27mm, F.Cu at (73.3, 44.3)
- added U2: Si4735-D60-GU, Package_SO:SSOP-24_3.9x8.7mm_P0.635mm, F.Cu at (65.1, 46.1)
- added U3: GVA-84+, Package_TO_SOT_SMD:SOT-89-3_Handsoldering, F.Cu at (73.5, 50.6)
- added U4: L7805CV, digikey-footprints:TO-220-3, F.Cu at (64.4, 37.9)
Other:
- board outline added: 101.6 x 69.9 mm

Commit message: Begin populating board
Parts:
- removed J4: Conn_01x07, Connector_PinHeader_2.54mm:PinHeader_1x07_P2.54mm_Vertical
- added C27: 0.1UF, Capacitor_SMD:C_0603_1608Metric, F.Cu at (177.0, 116.8)
- added C28: 0.1UF, Capacitor_SMD:C_0603_1608Metric, F.Cu at (193.0, 106.7)
- added C29: 0.1UF, Capacitor_SMD:C_0603_1608Metric, F.Cu at (187.2, 101.6)
- added C30: 0.1UF, Capacitor_SMD:C_0603_1608Metric, F.Cu at (182.1, 104.9)
- added IC1: SI5351C-B-GM1, SI5351C-B-GM1:QFN50P300X300X90-17N-D, F.Cu at (187.2, 105.6)
- added Y1: ASTX-H11-25.000MHZ-T, ASTX_H11_25_000MHZ_T:XTAL_ASTX-H11-25.000MHZ-T, F.Cu at (176.8, 110.6)
- J1: value HX8357D -> HX8357D SPI
- J5: value HX8357D -> HX8357D 8-BIT
- moved C26 165.3 mm to (193.0, 65.1), turned to 90 degrees
- moved C8 165.1 mm to (193.0, 58.4), turned to 90 degrees
- moved C10 164.8 mm to (193.0, 79.7), turned to 90 degrees
- moved C9 164.7 mm to (193.0, 72.7), turned to 90 degrees
- moved C20 153.4 mm to (193.0, 101.6), turned to 90 degrees
- moved C19 144.7 mm to (187.2, 81.3)
- moved Q3 143.2 mm to (175.3, 83.8), turned to -90 degrees
- moved Q4 142.7 mm to (175.3, 68.6), turned to 90 degrees
- moved C6 141.7 mm to (169.2, 78.7)
- moved C2 141.1 mm to (169.2, 66.0)
- moved C11 141.1 mm to (179.6, 81.3)
- moved C4 135.1 mm to (174.5, 61.0)
- moved L3 135.0 mm to (175.3, 96.5), turned to 90 degrees
- moved C1 130.0 mm to (169.4, 61.0)
- moved C14 129.0 mm to (166.9, 53.3), turned to 180 degrees
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Connections:
- C19 pad 1: /XMIT -> Net-(C19-Pad1)
- C21 pad 2: /XMIT -> Net-(C19-Pad1)
- J1 pad 1: (no net) -> unconnected-(J1-CD-Pad1)
- J1 pad 10: (no net) -> /Y+
- J1 pad 11: (no net) -> unconnected-(J1-LITE-Pad11)
- J1 pad 12: (no net) -> Net-(J1-RST)
- J1 pad 13: (no net) -> Net-(J1-D/C)
- J1 pad 14: (no net) -> Net-(J1-CS)
- J1 pad 15: (no net) -> /MOSI
- J1 pad 16: (no net) -> /MISO
- J1 pad 17: (no net) -> /DCLK
- J1 pad 18: (no net) -> Net-(J1-3Vo)
- J1 pad 19: (no net) -> +5V
- J1 pad 2: (no net) -> unconnected-(J1-CCS-Pad2)
- J1 pad 20: (no net) -> GND
- J1 pad 3: (no net) -> unconnected-(J1-IM0-Pad3)
- J1 pad 4: (no net) -> unconnected-(J1-IM1-Pad4)
- J1 pad 5: (no net) -> Net-(J1-3Vo)
- J1 pad 6: (no net) -> GND
- J1 pad 7: (no net) -> /X-
- J1 pad 8: (no net) -> /Y-
- J1 pad 9: (no net) -> /X+
- L3 pad 2: /XMIT -> Net-(C19-Pad1)
- TN1 pad 10: Net-(J1-Pin_12) -> Net-(J1-RST)
- TN1 pad 11: Net-(J1-Pin_13) -> Net-(J1-D/C)
- TN1 pad 12: Net-(J1-Pin_14) -> Net-(J1-CS)
- U3 pad 3: /XMIT -> Net-(C19-Pad1)

Commit message: Commit ongoing component placement
Parts:
- moved C5 142.9 mm to (168.9, 68.3), turned to 90 degrees
- moved C3 136.1 mm to (175.3, 68.1), turned to 90 degrees
- moved C27 14.9 mm to (191.8, 115.1), turned to 90 degrees
- moved C2 13.0 mm to (168.9, 79.1), turned to -90 degrees
- moved Y1 11.3 mm to (187.0, 115.5)
- moved BAT1 9.16 mm to (121.9, 94.0), turned to -90 degrees
- moved TN1 8.13 mm to (146.8, 82.5)
- moved C19 8.08 mm to (193.0, 86.9), turned to 90 degrees
- moved U1 7.71 mm to (126.9, 56.5)
- moved C12 7.71 mm to (118.5, 56.5)
- moved Q4 7.62 mm to (175.3, 76.2)
- moved C6 7.31 mm to (168.9, 86.0), turned to -90 degrees
- moved C11 5.02 mm to (184.2, 83.3), turned to 90 degrees
- moved L3 4.58 mm to (179.1, 99.1)
- moved C30 3.95 mm to (180.3, 108.4)
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
Commit message: All components initially placed
Parts:
- removed C16, C17, C18, C21: 0.1UF, Capacitor_SMD:C_0603_1608Metric
- moved C15 156.1 mm to (193.0, 108.7), turned to 90 degrees
- moved Q1 147.7 mm to (168.9, 116.8), turned to 90 degrees
- moved Q2 142.9 mm to (168.9, 108.0), turned to 90 degrees
- moved C7 140.8 mm to (168.9, 74.6), turned to 90 degrees
- moved R7 130.6 mm to (180.3, 70.7), turned to 90 degrees
- moved R11 130.4 mm to (174.4, 108.8), turned to -90 degrees
- moved R2 125.6 mm to (168.9, 94.8), turned to -90 degrees
- moved R8 124.0 mm to (160.0, 117.7), turned to -90 degrees
- moved C22 123.5 mm to (163.8, 100.3), turned to 90 degrees
- moved R1 121.4 mm to (163.8, 94.8), turned to -90 degrees
- moved R9 120.0 mm to (160.0, 111.3), turned to 90 degrees
- moved R6 119.2 mm to (168.9, 82.1), turned to 90 degrees
- moved R10 116.5 mm to (160.0, 105.0), turned to 90 degrees
- moved R3 116.4 mm to (163.8, 67.3), turned to -90 degrees
- moved R4 112.1 mm to (163.8, 82.1), turned to 90 degrees
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
Commit message: Poured GND and 3.3V into zones on in.1 and in.2 layers
Routing:
- added copper zone on In2.Cu, net +3.3V
- added copper zone on In1.Cu, net GND
Changed lines of the file:
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@@
 		(tags "LED diameter 5.0mm 2 pins")
 		(property "Reference" "D1"
-			(at 1.27 -3.96 360)
+			(at 1.27 -3.96 0)
 			(layer "F.SilkS")
 			(effects
@@
 		)
 		(property "Value" "XMIT"
-			(at 1.27 3.96 360)
+			(at 1.27 3.96 0)
 			(layer "F.Fab")
 			(effects
@@
 		)
 		(fp_text user "${REFERENCE}"
-			(at 1.25 0 360)
+			(at 1.25 0 0)
 			(layer "F.Fab")
 			(effects
@@
 			(extension_offset 0.5) keep_text_aligned)
 	)
+	(zone
+		(net 2)
+		(net_name "GND")
+		(layer "In1.Cu")
+		(name "Ground Plane")
+		(hatch edge 0.5)
+		(connect_pads
+			(clearance 0.5)
+		)
+		(min_thickness 0.25)
+		(filled_areas_thickness no)
+		(fill yes
+			(thermal_gap 0.5)
+			(thermal_bridge_width 0.5)
+		)
+		(polygon
+			(pts
+				(xy 101.6 50.8) (xy 203.2 50.8) (xy 203.2 120.65) (xy 101.6 120.65)
+			)
+		)
+	)
+	(zone
+		(net 3)
+		(net_name "+3.3V")
+		(layer "In2.Cu")
+		(name "PWR +3.3V")
+		(hatch edge 0.5)
+		(priority 1)
+		(connect_pads
+			(clearance 0.5)
+		)
+		(min_thickness 0.25)
+		(filled_areas_thickness no)
+		(fill yes
+			(thermal_gap 0.5)
+			(thermal_bridge_width 0.5)
+		)
+		(polygon
+			(pts
+				(xy 101.6 50.8) (xy 203.2 50.8) (xy 203.2 120.65) (xy 101.6 120.65)
+			)
+		)
+	)
 )

Commit message: routin in progress
Parts:
- moved C12 5.08 mm to (121.9, 64.3), turned to -90 degrees
- moved TN1 1.37 mm to (147.3, 83.8)
- moved C24 1.27 mm to (125.7, 73.2)
- moved C25 1.26 mm to (135.9, 89.4)
- moved C23 0.22 mm to (116.8, 64.5)
Routing:
- net +5V: track 0.00 -> 150.0 mm, vias 0 -> 1
- net /SDA: track 0.00 -> 115.9 mm, vias 0 -> 2
- net /Y+: track 0.00 -> 75.6 mm, vias 0 -> 2
- net /X-: track 0.00 -> 71.3 mm, vias 0 -> 2
- net GND: track 0.00 -> 51.6 mm, vias 0 -> 6
- net Net-(TN1-VBAT): track 0.00 -> 46.1 mm, vias 0 -> 2
- net /SCL: track 0.00 -> 39.1 mm
- net +12V: track 0.00 -> 17.8 mm
- net +3.3V: track 0.00 -> 14.8 mm, vias 0 -> 2

Commit message: Routing in progress
Parts:
- removed C22, C30: 0.1UF, Capacitor_SMD:C_0603_1608Metric
- removed REF** (x4): MountingHole_2.2mm_M2, MountingHole:MountingHole_2.2mm_M2
- moved C27 6.48 mm to (182.9, 116.3)
- moved Y1 4.13 mm to (188.5, 116.5), turned to 90 degrees
- moved R8 3.42 mm to (162.6, 115.4)
- moved C29 3.25 mm to (186.9, 104.0)
- moved C11 1.91 mm to (184.2, 85.2)
- moved U3 1.29 mm to (190.5, 92.7)
- moved L3 0.81 mm to (179.1, 98.2)
- moved Q1 0.63 mm to (168.9, 117.5)
- moved U2 0.32 mm to (172.4, 55.9)
- turned C5 to -90 degrees
- turned R2 to 90 degrees
Connections:
- C28 pad 1: Net-(IC1-VDD) -> +3.3V
- C29 pad 2: Net-(IC1-VDD) -> +3.3V
- IC1 pad 11: Net-(IC1-VDD) -> +3.3V
- IC1 pad 14: Net-(IC1-VDD) -> +3.3V
- IC1 pad 16: Net-(IC1-VDD) -> +3.3V
- IC1 pad 8: Net-(IC1-VDD) -> +3.3V
- IC1 pad 9: Net-(IC1-VDD) -> +3.3V
Routing:
- net /SCL: track 39.1 -> 110.7 mm, vias 0 -> 5
- net /MOSI: track 0.00 -> 69.7 mm, vias 0 -> 3
- net Net-(J1-CS): track 0.00 -> 68.9 mm, vias 0 -> 2
- net /X-: track 71.3 -> 140.0 mm, vias 2 -> 5
- net /MISO: track 0.00 -> 68.2 mm, vias 0 -> 2
- net /Y-: track 0.00 -> 68.1 mm, vias 0 -> 2
- net /Y+: track 75.6 -> 138.0 mm, vias 2 -> 5
- net /RCLK: track 0.00 -> 61.2 mm, vias 0 -> 2
- net /DCLK: track 0.00 -> 59.4 mm, vias 0 -> 2
- net /X+: track 0.00 -> 57.9 mm, vias 0 -> 4
- net +5V: track 150.0 -> 200.5 mm, vias 1 -> 3
- net /RECV: track 0.00 -> 49.1 mm, vias 0 -> 1
- net Net-(J1-3Vo): track 0.00 -> 35.3 mm
- net /SDA: track 115.9 -> 143.8 mm, vias 2 -> 5
- net +3.3V: track 14.8 -> 39.3 mm, vias 2 -> 8
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
Commit message: Routing in progress
Parts:
- moved R4 2.03 mm to (163.8, 80.1)
- moved R5 1.91 mm to (163.8, 86.5)
- moved R6 1.78 mm to (168.9, 80.3)
- moved C5 1.78 mm to (168.9, 86.8)
- moved L3 1.14 mm to (180.2, 98.2)
- moved C19 0.62 mm to (192.9, 86.2)
- moved C14 0.53 mm to (163.8, 54.4), turned to 90 degrees
- moved C10 0.13 mm to (192.9, 79.7)
- turned C9 to -90 degrees
Routing:
- net Net-(J1-RST): track 0.00 -> 69.0 mm, vias 0 -> 2
- net Net-(J1-D/C): track 0.00 -> 68.2 mm, vias 0 -> 2
- net GND: track 58.3 -> 97.5 mm, vias 16 -> 24
- net Net-(Q3-S): track 0.00 -> 29.2 mm, vias 0 -> 1
- net /XMIT: track 18.2 -> 46.4 mm
- net +3.3V: track 39.3 -> 66.1 mm, vias 8 -> 9
- net Net-(C26-Pad1): track 0.00 -> 23.5 mm
- net Net-(C7-Pad2): track 0.00 -> 23.2 mm, vias 0 -> 2
- net Net-(J2-ANT): track 0.00 -> 19.3 mm
- net Net-(C10-Pad1): track 0.00 -> 18.1 mm
- net Net-(TN1-16_A2_RX4_SCL1): track 0.00 -> 13.7 mm
- net Net-(C2-Pad2): track 0.00 -> 10.8 mm
- net Net-(Q3-D): track 0.00 -> 10.5 mm, vias 0 -> 1
- net +5V: track 200.5 -> 209.8 mm
- net Net-(C19-Pad1): track 18.0 -> 17.4 mm
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