File: hw/PocketFT8Xcvr.kicad_sch (KiCad schematic)
At the start: 57 parts, among them IC1 SI5351C-B-GM1, J1 HX8357D SPI, J2 22-23-2021, J3 22-23-2021, J5 HX8357D 8-BIT, Q1 2N3904, Q2 2N3906, Q3 2N7000, Q4 2N7000, U1 MCP3422A1T-E/SN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

Commit message: routin in progress
Parts:
- U4: now not fitted; now left out of the parts list
Changed lines of the file:
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@@
 				)
 				(justify left top)
+				(hide yes)
 			)
 		)
@@
 		(unit 1)
 		(exclude_from_sim no)
-		(in_bom yes)
+		(in_bom no)
 		(on_board yes)
-		(dnp no)
+		(dnp yes)
 		(fields_autoplaced yes)
 		(property "Reference" "U4"

Commit message: Routing in progress
Parts:
- removed C22, C30: 0.1UF, Capacitor_SMD:C_0603_1608Metric, symbol Kemet2024-08-02_22-05-35:C0603C104K4RACTU
Connections:
- net +3.3V: now also C28.1, C29.2, IC1.11 (VDDOD), IC1.14 (VDDOC), IC1.16 (VDD), IC1.8 (VDDOB), IC1.9 (VDDOA)

Commit message: Delete 7805 voltage regulator
Decision:  Avoid heat dissipation issues with 12->5V linear regulators through use of widely available portable USB power banks supplying 5V at >= 1A via a USB-C to MicroUSB-B cable.  These consumer devices deliver enough highly portable power for QRP communications.  Their external noise problems may be easier to resolve than the internal heat/noise problems of 5V regulator designs.  Long-term, "true" USB-C offers even more power capability should Teensy adopt it.
Parts:
- removed C23: 0.33UF, 0805, symbol Kemet2024-08-02_22-55-33:C0805C334K4RAC7800
- removed C24: 0.1UF, Capacitor_SMD:C_0603_1608Metric, symbol Kemet2024-08-02_22-05-35:C0603C104K4RACTU
- removed J3: 22-23-2021, digikey-footprints:PinHeader_1x2_P2.54mm_Drill1.02mm, symbol dk_Rectangular-Connectors-Headers-Male-Pins:22-23-2021
- removed U4: L7805CV, TO-220-3, symbol dk_PMIC-Voltage-Regulators-Linear:L7805CV
Connections:
- net +5V: no longer TN1.48 (VIN)

Commit message: Add GPS connector to schematic
Parts:
- added J3: GPS, digikey-footprints:PinHeader_1x4_P2.54mm_Drill1.02mm, symbol dk_Rectangular-Connectors-Headers-Male-Pins:0022232041
Connections:
- no-connect marks 81 -> 79
Other:
- moved on the sheet: C12, U1

Commit message: Added GPS connector to board
Parts:
- J3: now not fitted; now left out of the parts list
Connections:
- net +3.3V: now also J3.4 (+3.3V)
- net GND: now also J3.1 (GND)
- net GPSTX: now reaches J3.2 (GPSTX)
- net GPSTX: now also TN1.2 (0_RX1_CRX2_CS1)
- net GPSRX: now reaches J3.3 (GPSRX)
- net GPSRX: now also TN1.3 (1_TX1_CTX2_MISO1)
Changed lines of the file:
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@@
 	)
 	(junction
-		(at 96.52 44.45)
+		(at 85.36 44.45)
 		(diameter 0)
 		(color 0 0 0 0)
@@
 	)
 	(junction
+		(at 91.44 44.45)
+		(diameter 0)
+		(color 0 0 0 0)
+	)
+	(junction
 		(at 264.16 142.24)
 		(diameter 0)
@@
 	)
 	(junction
+		(at 85.36 52.07)
+		(diameter 0)
+		(color 0 0 0 0)
+	)
+	(junction
 		(at 214.63 33.02)
 		(diameter 0)
@@
 	)
 	(junction
+		(at 85.36 49.53)
+		(diameter 0)
+		(color 0 0 0 0)
+	)
+	(junction
 		(at 207.01 109.22)
 		(diameter 0)
@@
 	)
 	(junction
+		(at 85.36 46.99)
+		(diameter 0)
+		(color 0 0 0 0)
+	)
+	(junction
 		(at 162.56 40.64)
 		(diameter 0)
@@
 	(wire
 		(pts
+			(xy 91.44 44.45) (xy 104.14 44.45)
+		)
+		(stroke
+			(width 0)
+			(type default)
+		)
+	)
+	(wire
+		(pts
 			(xy 34.29 67.31) (xy 104.14 67.31)
 		)
@@
 	(wire
 		(pts
-			(xy 96.52 44.45) (xy 104.14 44.45)
-		)
-		(stroke
-			(width 0)
-			(type default)
-		)
-	)
-	(wire
-		(pts
 			(xy 232.41 93.98) (xy 238.76 93.98)
 		)
@@
 	(wire
 		(pts
-			(xy 85.09 46.99) (xy 104.14 46.99)
+			(xy 85.09 46.99) (xy 85.36 46.99)
 		)
 		(stroke
@@
 	(wire
 		(pts
-			(xy 85.09 49.53) (xy 104.14 49.53)
+			(xy 85.09 49.53) (xy 85.36 49.53)
 		)
 		(stroke
@@
 	(wire
 		(pts
+			(xy 85.36 52.07) (xy 85.09 52.07)
+		)
+		(stroke
+			(width 0)
+			(type default)
+		)
+	)
+	(wire
+		(pts
 			(xy 207.01 142.24) (xy 212.09 142.24)
 		)
@@
 	(wire
 		(pts
+			(xy 85.36 44.45) (xy 91.44 44.45)
+		)
+		(stroke
+			(width 0)
+			(type default)
+		)
+	)
+	(wire
+		(pts
 			(xy 115.57 163.83) (xy 115.57 167.64)
 		)
@@
 	(wire
 		(pts
+			(xy 85.36 49.53) (xy 104.14 49.53)
+		)
+		(stroke
+			(width 0)
+			(type default)
+		)
+	)
+	(wire
+		(pts
 			(xy 97.79 80.01) (xy 104.14 80.01)
 		)
@@
 	(wire
 		(pts
+			(xy 85.36 46.99) (xy 104.14 46.99)
+		)
+		(stroke
+			(width 0)
+			(type default)
+		)
+	)
+	(wire
+		(pts
 			(xy 279.4 119.38) (xy 279.4 149.86)
 		)
@@
 	(wire
 		(pts
-			(xy 85.09 44.45) (xy 96.52 44.45)
+			(xy 85.09 44.45) (xy 85.36 44.45)
 		)
 		(stroke
@@
 	(wire
 		(pts
-			(xy 91.44 52.07) (xy 85.09 52.07)
+			(xy 91.44 52.07) (xy 85.36 52.07)
 		)
 		(stroke
@@
 		)
 	)
+	(label "GPSTX"
+		(at 97.79 46.99 0)
+		(fields_autoplaced yes)
+		(effects
+			(font
+				(size 1.27 1.27)
+			)
+			(justify left bottom)
+		)
+	)
 	(label "DCLK"
 		(at 57.15 21.59 0)
@@
 		)
 	)
+	(label "GPSRX"
+		(at 97.79 49.53 0)
+		(fields_autoplaced yes)
+		(effects
+			(font
+				(size 1.27 1.27)
+			)
+			(justify left bottom)
+		)
+	)
 	(label "PTT"
 		(at 160.02 77.47 0)
@@
 	(symbol
 		(lib_id "power:GND")
-		(at 96.52 44.45 180)
+		(at 91.44 44.45 180)
 		(unit 1)
 		(exclude_from_sim no)
@@
 		(fields_autoplaced yes)
 		(property "Reference" "#PWR08"
-			(at 96.52 38.1 0)
+			(at 91.44 38.1 0)
 			(effects
 				(font
@@
 		)
 		(property "Value" "GND"
-			(at 99.06 43.1799 0)
+			(at 93.98 43.1799 0)
 			(effects
 				(font
@@
 		)
 		(property "Footprint" ""
-			(at 96.52 44.45 0)
+			(at 91.44 44.45 0)
 			(effects
 				(font
@@
 		)
 		(property "Datasheet" ""
-			(at 96.52 44.45 0)
+			(at 91.44 44.45 0)
 			(effects
 				(font
@@
 		)
 		(property "Description" "Power symbol creates a global label with name \"GND\" , ground"
-			(at 96.52 44.45 0)
+			(at 91.44 44.45 0)
 			(effects
 				(font
@@
 	(symbol
 		(lib_id "dk_Rectangular-Connectors-Headers-Male-Pins:0022232041")
-		(at 82.55 44.45 270)
+		(at 83.82 44.45 270)
 		(unit 1)
 		(exclude_from_sim no)
-		(in_bom yes)
+		(in_bom no)
 		(on_board yes)
-		(dnp no)
+		(dnp yes)
 		(fields_autoplaced yes)
 		(property "Reference" "J3"
-			(at 81.28 38.1 90)
+			(at 82.55 38.1 90)
 			(effects
 				(font
@@
 		)
 		(property "Value" "GPS"
-			(at 81.28 40.64 90)
+			(at 82.55 40.64 90)
 			(effects
 				(font
@@
 		)
 		(property "Footprint" "digikey-footprints:PinHeader_1x4_P2.54mm_Drill1.02mm"
-			(at 87.63 49.53 0)
+			(at 88.9 49.53 0)
 			(effects
 				(font
@@
 		)
 		(property "Datasheet" "https://www.molex.com/pdm_docs/sd/022232041_sd.pdf"
-			(at 90.17 49.53 0)
+			(at 91.44 49.53 0)
 			(effects
 				(font
@@
 		)
 		(property "Description" "CONN HEADER VERT 4POS 2.54MM"
-			(at 82.55 44.45 0)
+			(at 83.82 44.45 0)
 			(effects
 				(font
@@
 		)
 		(property "Digi-Key_PN" "WM4202-ND"
-			(at 92.71 49.53 0)
+			(at 93.98 49.53 0)
 			(effects
 				(font
@@
 		)
 		(property "MPN" "0022232041"
-			(at 95.25 49.53 0)
+			(at 96.52 49.53 0)
 			(effects
 				(font
@@
 		)
 		(property "Category" "Connectors, Interconnects"
-			(at 97.79 49.53 0)
+			(at 99.06 49.53 0)
 			(effects
 				(font
@@
 		)
 		(property "Family" "Rectangular Connectors - Headers, Male Pins"
-			(at 100.33 49.53 0)
+			(at 101.6 49.53 0)
 			(effects
 				(font
@@
 		)
 		(property "DK_Datasheet_Link" "https://www.molex.com/pdm_docs/sd/022232041_sd.pdf"
-			(at 102.87 49.53 0)
+			(at 104.14 49.53 0)
 			(effects
 				(font
@@
 		)
 		(property "DK_Detail_Page" "/product-detail/en/molex/0022232041/WM4202-ND/26671"
-			(at 105.41 49.53 0)
+			(at 106.68 49.53 0)
 			(effects
 				(font
@@
 		)
 		(property "Description_1" "CONN HEADER VERT 4POS 2.54MM"
-			(at 107.95 49.53 0)
+			(at 109.22 49.53 0)
 			(effects
 				(font
@@
 		)
 		(property "Manufacturer" "Molex"
-			(at 110.49 49.53 0)
+			(at 111.76 49.53 0)
 			(effects
 				(font
@@
 		)
 		(property "Status" "Active"
-			(at 113.03 49.53 0)
+			(at 114.3 49.53 0)
 			(effects
 				(font

Commit message: Review-1
Parts:
- added C16, C17: 0.1UF, Capacitor_SMD:C_0603_1608Metric, symbol Kemet2024-08-02_22-05-35:C0603C104K4RACTU
Connections:
- net +5V: now also C17.2
- net GND: now also C16.1, C17.1
- net XMIT: now also C16.2

Commit message: Clean DRC
Connections:
- no-connect marks 79 -> 80
Changed lines of the file:
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@@
-	)
-	(junction
-		(at 85.36 44.45)
-		(diameter 0)
-		(color 0 0 0 0)
 	)
 	(junction
@@
 	)
 	(junction
-		(at 85.36 52.07)
-		(diameter 0)
-		(color 0 0 0 0)
-	)
-	(junction
 		(at 214.63 33.02)
 		(diameter 0)
@@
 	)
 	(junction
-		(at 85.36 49.53)
-		(diameter 0)
-		(color 0 0 0 0)
-	)
-	(junction
 		(at 207.01 109.22)
 		(diameter 0)
@@
 	)
 	(junction
-		(at 85.36 46.99)
-		(diameter 0)
-		(color 0 0 0 0)
-	)
-	(junction
 		(at 162.56 40.64)
 		(diameter 0)
@@
 	)
 	(no_connect
+		(at 160.02 44.45)
+	)
+	(no_connect
 		(at 78.74 172.72)
 	)
@@
 	(wire
 		(pts
-			(xy 85.09 46.99) (xy 85.36 46.99)
+			(xy 85.09 46.99) (xy 104.14 46.99)
 		)
 		(stroke
@@
 	(wire
 		(pts
-			(xy 85.09 49.53) (xy 85.36 49.53)
+			(xy 85.09 49.53) (xy 104.14 49.53)
 		)
 		(stroke
@@
 	(wire
 		(pts
-			(xy 85.36 52.07) (xy 85.09 52.07)
+			(xy 85.09 52.07) (xy 91.44 52.07)
 		)
 		(stroke
@@
 	(wire
 		(pts
-			(xy 85.36 44.45) (xy 91.44 44.45)
-		)
-		(stroke
-			(width 0)
-			(type default)
-		)
-	)
-	(wire
-		(pts
 			(xy 115.57 163.83) (xy 115.57 167.64)
 		)
@@
 	(wire
 		(pts
-			(xy 85.36 49.53) (xy 104.14 49.53)
-		)
-		(stroke
-			(width 0)
-			(type default)
-		)
-	)
-	(wire
-		(pts
 			(xy 97.79 80.01) (xy 104.14 80.01)
 		)
@@
 	(wire
 		(pts
-			(xy 85.36 46.99) (xy 104.14 46.99)
-		)
-		(stroke
-			(width 0)
-			(type default)
-		)
-	)
-	(wire
-		(pts
 			(xy 279.4 119.38) (xy 279.4 149.86)
 		)
@@
 	(wire
 		(pts
-			(xy 85.09 44.45) (xy 85.36 44.45)
+			(xy 85.09 44.45) (xy 91.44 44.45)
 		)
 		(stroke
@@
 		)
 		(stroke
-			(width 0)
-			(type default)
-		)
-	)
-	(wire
-		(pts
-			(xy 91.44 52.07) (xy 85.36 52.07)
-		)
-		(stroke

Commit message: Minor cleanup
Parts:
- IC1: Manufacturer (none) -> Skyworks; Manufacturer_Name Skyworks -> (none)
- R6: Manufacturer YAGEO -> Yageo
- Y1: MANUFACTURER Abracon -> (none); Manufacturer (none) -> Abracon; Mfg Part # (none) -> ASTX-H11-25.000MHZ-T; Type (none) -> SMD
Connections:
- net +3.3V: now also TN1.51 (3V3)
- net GND: now also TN1.52 (GND)
- no-connect marks 80 -> 78
Other:
- moved on the sheet: BAT1
