File: Investigations/LowPassFilter2ndHarmonicTrap/LowPassFilter.kicad_sch (KiCad schematic)
At the start: 9 parts

Commit message: Simulations of Low Pass Filter + Harmonic Trap
Parts:
- C1: value 243pf -> 430 pF
- C2: value 75pf -> 130 pF
- C3: renamed from C4; value 52pf -> 44 pF
- C4: renamed from C3; value 75pf -> 130 pF
- L1: value 0.5 uh -> 0.910 uH
- L2: value .375uh -> .683 uH
