File: PocketFT8XcvrHWQFN20/PocketFT8Xcvr.kicad_pcb (KiCad board)
At the start: 4 copper layers, 101.6 x 69.9 mm, 58 parts, among them J1 HX8357D SPI, J2 22-23-2021, J3 GPS, J5 HX8357D 8-BIT, Q1 2N3904, Q2 2N3906, Q3 2N7000, Q4 2N7000, U1 MCP3422A1T-E/SN, U2 Si4735-D60-GU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

Commit message: Resubmit to PCBWay with SI5351c QFN20 Package
QFN16 was unobtanium
Changed lines of the file:
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@@
 		(pad_to_mask_clearance 0)
 		(allow_soldermask_bridges_in_footprints no)
+		(aux_axis_origin 101.6 120.65)
+		(grid_origin 101.6 120.65)
 		(pcbplotparams
 			(layerselection 0x00010fc_ffffffff)
@@
 			(disableapertmacros no)
 			(usegerberextensions no)
-			(usegerberattributes yes)
-			(usegerberadvancedattributes yes)
-			(creategerberjobfile yes)
+			(usegerberattributes no)
+			(usegerberadvancedattributes no)
+			(creategerberjobfile no)
 			(dashed_line_dash_ratio 12.000000)
 			(dashed_line_gap_ratio 3.000000)
@@
 			(psa4output no)
 			(plotreference yes)
-			(plotvalue yes)
+			(plotvalue no)
 			(plotfptext yes)
 			(plotinvisibletext no)
 			(sketchpadsonfab no)
-			(subtractmaskfromsilk no)
+			(subtractmaskfromsilk yes)
 			(outputformat 1)
 			(mirror no)
-			(drillshape 1)
+			(drillshape 0)
 			(scaleselection 1)
-			(outputdirectory "")
+			(outputdirectory "./CAM")
 		)
 	)
@@
 		(tags "SI5351C-B-GM ")
 		(property "Reference" "U4"
-			(at -3.576828 2.6543 0)
+			(at 0 0 0)
 			(unlocked yes)
 			(layer "F.SilkS")
@@
 			(unlocked yes)
 			(layer "F.Fab")
-			(hide yes)
 			(effects
 				(font
@@
 			)
 		)
-		(property "Footprint" "SI5351C-B-GM:QFN20_4X4_SKY"
+		(property "Footprint" "QFN20_4X4_SKY"
 			(at 0 0 0)
 			(layer "F.Fab")
@@
 			)
 		)
-		(property "Description" ""
+		(property "Description" "IC CLOCK GENERATOR 20QFN"
 			(at 0 0 0)
 			(layer "F.Fab")
@@
 			)
 		)
+		(property "Manufacturer" "Skyworks Solutions"
+			(at 0 0 0)
+			(unlocked yes)
+			(layer "F.Fab")
+			(hide yes)
+			(effects
+				(font
+					(size 1 1)
+					(thickness 0.15)
+				)
+			)
+		)
+		(property "Mfg Part #" "SI5351C-B-GM"
+			(at 0 0 0)
+			(unlocked yes)
+			(layer "F.Fab")
+			(hide yes)
+			(effects
+				(font
+					(size 1 1)
+					(thickness 0.15)
+				)
+			)
+		)
+		(property "Type" "SMT"
+			(at 0 0 0)
+			(unlocked yes)
+			(layer "F.Fab")
+			(hide yes)
+			(effects
+				(font
+					(size 1 1)
+					(thickness 0.15)
+				)
+			)
+		)
+		(property "Notes" "https://www.digikey.com/en/products/detail/skyworks-solutions-inc/SI5351C-B-GM/3679850"
+			(at 0 0 0)
+			(unlocked yes)
+			(layer "F.Fab")
+			(hide yes)
+			(effects
+				(font
+					(size 1 1)
+					(thickness 0.15)
+				)
+			)
+		)
 		(property ki_fp_filters "QFN20_4X4_SKY QFN20_4X4_SKY-M QFN20_4X4_SKY-L")
 		(sheetname "Root")
 		(sheetfile "PocketFT8Xcvr.kicad_sch")
-		(clearance 0.15)
 		(attr smd)
 		(fp_poly
@@
 		(fp_text user "*"
 			(at -2.9337 -1.243965 0)
-			(unlocked yes)
 			(layer "F.SilkS")
 			(effects
@@
 		(fp_text user "*"
 			(at -1.5367 -1.243965 0)
-			(unlocked yes)
 			(layer "F.Fab")
 			(effects
@@
 			)
 		)
-		(fp_text user "${REFERENCE}"
-			(at 0 0 0)
+		(fp_text user "*"
+			(at -1.5367 -1.243965 0)
 			(unlocked yes)
 			(layer "F.Fab")
@@
 			)
 		)
-		(fp_text user "*"
-			(at -1.5367 -1.243965 0)
+		(fp_text user "${REFERENCE}"
+			(at 0 0 0)
 			(unlocked yes)
 			(layer "F.Fab")
@@
 		)
 		(height -12.7)
-		(gr_text "2.4000 in"
+		(gr_text "60.9600 mm"
 			(at 209.02 84.455 90)
 			(layer "Cmts.User")
@@
 		)
 		(height -8.255)
-		(gr_text "3.6000 in"
+		(gr_text "91.4400 mm"
 			(at 152.908 43.942 0)
 			(layer "Cmts.User")
