File: PocketFT8XcvrHWQFN20/PocketFT8Xcvr.kicad_sch (KiCad schematic)
At the start: 54 parts, among them J1 HX8357D SPI, J2 22-23-2021, J3 GPS, J5 HX8357D 8-BIT, Q1 2N3904, Q2 2N3906, Q3 2N7000, Q4 2N7000, U1 MCP3422A1T-E/SN, U2 Si4735-D60-GU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

Commit message: Resubmit to PCBWay with SI5351c QFN20 Package
QFN16 was unobtanium
Parts:
- U4: Manufacturer (none) -> Skyworks Solutions; Mfg Part # (none) -> SI5351C-B-GM; Notes (none) -> https://www.digikey.com/en/products/detail/skyworks-solutio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; Type (none) -> SMT
