File: PocketFT8XcvrHW.old/PocketFT8Xcvr.kicad_pcb (KiCad board)
At the start: 4 copper layers, 101.6 x 69.9 mm, 58 parts, among them J1 HX8357D SPI, J2 22-23-2021, J3 GPS, J5 HX8357D 8-BIT, Q1 2N3904, Q2 2N3906, Q3 2N7000, Q4 2N7000, U1 MCP3422A1T-E/SN, U2 Si4735-D60-GU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

Commit message: Housecleaning after abandoning the QFN16 SI5351 package
Parts:
- removed U4: SI5351C-B-GM, SI5351C-B-GM:QFN20_4X4_SKY
- added IC1: SI5351C-B-GM1, SI5351C-B-GM1:QFN50P300X300X90-17N-D, F.Cu at (183.9, 108.7)
- moved C29 0.63 mm to (186.9, 104.0)
Routing:
- net +3.3V: track 79.9 -> 71.3 mm, vias 12 -> 10
- net /SDA: track 171.0 -> 178.1 mm
- net /RCLK: track 68.2 -> 61.2 mm
- net Net-(IC1-CLKIN): track 14.0 -> 9.17 mm
- net /SCL: track 137.2 -> 141.1 mm
- net GND: track 80.0 -> 80.7 mm, vias 32 -> 31
Other:
- board text removed: "KQ7B POCKET FT8 V1.00"
