File: Investigations/PAClassD/ClassDSimulation/ClassDSimulation.kicad_sch (KiCad schematic)
At the start: 17 parts, among them Q1 BS170, Q2 BS170

Commit message: Saving everything as Board Turn-On begins
Parts:
- added C5: 910p, SparkFun-Capacitor:C_0603_1608Metric, symbol SparkFun-Capacitor:C
- added L5: 1.2u, SparkFun-Capacitor:C_0805_2012Metric, symbol SparkFun-Coil:L
- C1: value 620 pF -> 910p
- C3: renamed from C2; value 620 pF -> 1300p
- L4: value 750 nH -> 1.2u
Connections:
- net GND: now also C5.2
- net Vo: now also C5.1, L5.2; no longer C3.1, L4.2
- net Vd1: now reaches L1.2, Q1.1 (D)
- new net: C3.1, L4.2, L5.1
Other:
- moved on the sheet: R1
