File: Investigations/PAClassE/PAClassE.kicad_sch (KiCad schematic)
At the start: 13 parts, among them Q1 BS170, Q2 BS170, Q3 BS170

Commit message: Class E hand tuned to C1=332pF
Parts:
- C1: value 360 p -> 368p
- C2: value 510 p -> 510p
- L2: value 1.28 u -> 1.28u
Changed lines of the file:
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@@
 		)
 	)
-	(text_box "Notes:  Ideal Class E tank capacitor values calculated by https://people.physics.anu.edu.au/~dxt103/calculators/class-e.php approximated here by standard capacitor values.\n\nTank circuit calculations performed for 3 paralleled BS170 transistors, Coss(parallel) = 51 pF.\n\nR4 inserted to simulate Q(L2).\n\nVPULSE and R1 approximate drive from 3 paralleled 74ACT00 gates.\n\nQ1, Q2 and Q3 paralleled to reduce their effective (paralleled) Rds for use with 5V supply.  Their paralleled Ciss ~= 85 pF.\n"
+	(text_box "Notes:  Ideal Class E tank capacitor values calculated by https://people.physics.anu.edu.au/~dxt103/calculators/class-e.php approximated here by standard capacitor values.\n\nTank circuit calculations performed for 3 paralleled BS170 transistors, Coss(parallel) = 51 pF.\n\nR4 inserted to simulate tank circuit Q.\n\nVPULSE and R1 approximate drive from 3 paralleled 74ACT00 gates.\n\nQ1, Q2 and Q3 paralleled to reduce their effective (paralleled) Rds for use with 5V supply.  Their paralleled Ciss ~= 85 pF.\n"
 		(exclude_from_sim no)
 		(at 121.92 102.87 0)
@@
 			)
 		)
-		(property "Value" "360 p"
+		(property "Value" "368p"
 			(at 119.38 81.2799 0)
 			(effects
@@
 				)
 				(justify left)
+			)
+		)
+		(property "Sim.Device" "C"
+			(at 0 165.1 0)
+			(effects
+				(font
+					(size 1.27 1.27)
+				)
+				(hide yes)
+			)
+		)
+		(property "Sim.Pins" "1=+ 2=-"
+			(at 0 165.1 0)
+			(effects
+				(font
+					(size 1.27 1.27)
+				)
+				(hide yes)
 			)
 		)
@@
 			)
 		)
-		(property "Value" "510 p"
+		(property "Value" "510p"
 			(at 123.19 63.5 90)
 			(effects
@@
 			)
 		)
-		(property "Value" "1.28 u"
+		(property "Value" "1.28u"
 			(at 143.51 71.12 0)
 			(effects

Commit message: Saving everything as Board Turn-On begins
Parts:
- L1: value 47 u -> 47u
- R3: value 12.5 -> 5.5
Changed lines of the file:
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@@
 			)
 		)
-		(property "Value" "47 u"
+		(property "Value" "47u"
 			(at 97.79 67.3099 90)
 			(effects
@@
 			)
 		)
-		(property "Value" "12.5"
+		(property "Value" "5.5"
 			(at 156.21 83.8199 0)
 			(effects
