File: PocketFT8Filters/PocketFT8Filters.kicad_sch (KiCad schematic)
At the start: 10 parts

Commit message: Ongoing filter daughter board development
Parts:
- removed C1, C2, C3, C4, C5: C, Capacitor_SMD:C_1206_3216Metric_Pad1.33x1.80mm_HandSolder, symbol Device:C
- removed L1, L2, L3, L4, L5: L_Ferrite, symbol Device:L_Ferrite
