File: PocketFT8XcvrHW/PocketFT8Xcvr.kicad_pcb (KiCad board)
At the start: 4 copper layers, 100 x 69.9 mm, 64 parts, among them J1 HX8357D SPI, J2 22-23-2021, J3 B5B-XH-A_LF__SN_, J5 HX8357D 8-BIT, Q1 2N7002DW, U1 MCP3422A1T-E/SN, U2 Si4735-D60-GU, U3 SN74ACT244DWR, U4 SI5351C-B-GM, Y1 ASTX-H11-25.000MHZ-T

Commit message: Preparing V2.00 board for fab
Parts:
- removed C1, C2, C4: 910pF, Capacitor_SMD:C_0805_2012Metric
- removed C3: 1300pF, Capacitor_SMD:C_0805_2012Metric
- removed L2, L3: 1.2uH, Inductor_THT:L_Toroid_Vertical_L10.0mm_W5.0mm_P5.08mm
- removed L4: L_Ferrite_Coupled, Inductor_THT:L_Toroid_Vertical_BIFILAR
- added FL1: ~, Filters:PluginFilter, F.Cu at (187.1, 79.8)
- added TP5: PTH, SparkFun-Connector:1x01, F.Cu at (166.3, 111.2)
- added TP6: PTH, SparkFun-Connector:1x01, F.Cu at (170.0, 111.3)
- J2: value 22-23-2021 -> CONN SMA JACK STR 50OHM EDGE MNT; footprint digikey-footprints:PinHeader_1x2_P2.54mm_Drill1.02mm -> digikey-footprints:RF_SMA_BoardEdge_142-0701-801
- L1: value 1.2uH -> L_Ferrite_Coupled; footprint Inductor_THT:L_Toroid_Vertical_L10.0mm_W5.0mm_P5.08mm -> Inductor_THT:L_Toroid_Vertical_BIFILAR
- R12, R13: value 510 -> 510 OHMS
- R5: value 2.2K -> 2.2K OHM
- R6: value 10k -> 10k OHM
- moved L1 23.5 mm to (185.9, 115.6)
- moved C23 6.24 mm to (175.3, 82.3), turned to -90 degrees
- moved J2 4.92 mm to (187.9, 50.9), turned to 0 degrees
- moved C20 3.92 mm to (178.3, 91.0)
- moved C27 1.01 mm to (111.9, 70.2)
- moved C10 1.00 mm to (178.4, 70.4)
Connections:
- C20 pad 2: Net-(C1-Pad1) -> Net-(FL1-IN)
- L1 pad 1: Net-(C1-Pad1) -> GND
- L1 pad 2: Net-(C2-Pad1) -> Net-(C19-Pad2)
Routing:
- net Net-(C1-Pad1): track 33.6 -> 0.00 mm
- net /RCV: track 70.5 -> 97.1 mm, vias 4 -> 5
- net Net-(FL1-IN): track 0.00 -> 20.2 mm
- net GND: track 75.0 -> 90.5 mm, vias 36 -> 67
- net Net-(C2-Pad1): track 14.0 -> 0.00 mm
- net Net-(C3-Pad1): track 13.5 -> 0.00 mm
- net /XMT: track 45.6 -> 57.0 mm
- net Net-(FL1-OUT): track 9.38 -> 13.5 mm
- net /XD+: track 66.0 -> 63.7 mm
- net +3.3V: track 70.9 -> 69.9 mm
- net Net-(Q1-D2): track 18.5 -> 17.9 mm
- net /YD-: vias 3 -> 1

Commit message: Cleanup V2.00 for fab
Parts:
- R12, R13: value 510 OHMS -> 510
- R5: value 2.2K OHM -> 2.2K
- R6: value 10k OHM -> 10k
- moved C13 4.29 mm to (159.6, 58.9)
- moved C14 4.28 mm to (159.6, 54.4)
- moved R2 2.68 mm to (163.8, 60.8)
- moved C30 1.40 mm to (133.4, 84.6), turned to -90 degrees
- moved C12 1.19 mm to (124.8, 60.5)
- moved R6 0.18 mm to (168.9, 80.1), turned to -90 degrees
- turned C7 to -90 degrees
Routing:
- net +3.3V: track 69.9 -> 54.2 mm, vias 8 -> 9
- net GND: track 90.5 -> 104.3 mm, vias 67 -> 65
- net +5V: track 249.8 -> 244.4 mm
- net Net-(C7-Pad2): track 23.2 -> 17.9 mm, vias 2 -> 0
- net /YD-: track 66.0 -> 64.0 mm
- net /SCL: track 37.9 -> 36.7 mm
- net /XCLK: track 35.1 -> 34.5 mm
Other:
- board text added: "KQ7B POCKET FT8 V2.00"
- board text removed: "KQ7B POCKET FT8 V1.10"

Commit message: Cleanup for V2.00 fab
Connections:
- net Net-(FL1-IN) renamed /RF
- net Net-(FL1-OUT) renamed /ANT

Commit message: V2.00 Submission to PCBWay
Connections:
- net Net-(U4-CLKIN) renamed /CLK

Commit message: Ongoing filter daughter board development
Changed lines of the file:
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@@
 			(layer "F.CrtYd")
+		)
+		(fp_text user "IN"
+			(at -16.256 -2.286 90)
+			(unlocked yes)
+			(layer "F.SilkS")
+			(effects
+				(font
+					(size 2.54 2.54)
+					(thickness 0.254)
+				)
+				(justify left bottom)
+			)
+		)
+		(fp_text user "GND"
+			(at 8.89 4.826 90)
+			(unlocked yes)
+			(layer "F.SilkS")
+			(effects
+				(font
+					(size 2.54 2.54)
+					(thickness 0.254)
+				)
+				(justify left bottom)
+			)
 		)
 		(fp_text user "GND"
@@
 			)
 		)
-		(fp_text user "IN"
-			(at -16.256 -2.286 90)
-			(unlocked yes)
-			(layer "F.SilkS")
-			(effects
-				(font
-					(size 2.54 2.54)
-					(thickness 0.254)
-				)
-				(justify left bottom)
-			)
-		)
 		(fp_text user "OUT"
 			(at 8.89 -2.286 90)
-			(unlocked yes)
-			(layer "F.SilkS")
-			(effects
-				(font
-					(size 2.54 2.54)
-					(thickness 0.254)
-				)
-				(justify left bottom)
-			)
-		)
-		(fp_text user "GND"
-			(at 8.89 4.826 90)
 			(unlocked yes)
 			(layer "F.SilkS")
@@
 		)
 		(pad "2" thru_hole circle
-			(at -18.034 5.08 90)
+			(at -17.78 5.08 90)
 			(size 1.524 1.524)
 			(drill 0.762)

Commit message: V2.01 Correct schematic for 51 ohm, C22 and C23 values
Problem found by PCBway
Parts:
- C22, C23: value 10nF -> 0.1uF

Commit message: SI5351 moved from Wire to Wire2 in V2.00 hardware
Parts:
- renumbered L1 to T1
Changed lines of the file:
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@@
 		(descr "L_Toroid, Vertical series, Radial, pin pitch=5.08mm, , length*width=10*5mm^2")
 		(tags "L_Toroid Vertical series Radial pin pitch 5.08mm  length 10mm width 5mm")
-		(property "Reference" "L1"
+		(property "Reference" "T1"
 			(at -0.52 7.5 0)
 			(layer "F.SilkS")
@@
 		)
 		(height 7)
-		(gr_text "2400.0000 mils"
+		(gr_text "60.9600 mm"
 			(at 98.27 84.9 90)
 			(layer "Cmts.User")
@@
 		)
 		(height -8.21)
-		(gr_text "3600.0026 mils"
+		(gr_text "91.4401 mm"
 			(at 152.608 43.846 0.06892533581)
 			(layer "Cmts.User")
