File: RFFilters/5Pole40MLPFilter/5PoleLPFilter.kicad_sch (KiCad schematic)
At the start: 5 parts

Commit message: Update 5PoleLP Filter
+ V4.00 Hardware LP Filter PCB
+ Remove deprecated files
Connections:
- net In: now reaches C1.1, L1.1
- net Mid: now reaches C2.1, L1.2, L2.1
- net Out: now reaches C3.1, L2.2
Changed lines of the file:
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@@
 (kicad_sch
-	(version 20231120)
+	(version 20250114)
 	(generator "eeschema")
-	(generator_version "8.0")
+	(generator_version "9.0")
 	(paper "A4")
 	(junction
@@
 			(width 0)
 			(type default)
+		)
+	)
+	(label "Mid"
+		(at 110.49 74.93 0)
+		(effects
+			(font
+				(size 1.27 1.27)
+			)
+			(justify left bottom)
+		)
+	)
+	(label "In"
+		(at 69.85 74.93 0)
+		(effects
+			(font
+				(size 1.27 1.27)
+			)
+			(justify left bottom)
+		)
+	)
+	(label "Out"
+		(at 149.86 74.93 0)
+		(effects
+			(font
+				(size 1.27 1.27)
+			)
+			(justify left bottom)
 		)
 	)
@@
 		)
 	)
+	(embedded_fonts no)
 )
